File: encoder.kicad_sch (KiCad schematic)
At the start: 1 part, among them J3 Conn_01x08

Commit message: PCB Finished, only have to check LED's
Parts:
- added C49: 100N-X7R_50V#0603, D&R_Passive:C_0603, symbol D&R_Passive:100N-X7R_50V#0603
- added R28, R29, R30: 120R#0603, D&R_Passive:R_0603, symbol D&R_Passive:120R#0603
- added U16: AM26LV32E, Package_SO:TSSOP-16_4.4x5mm_P0.65mm, symbol Doggen:AM26LV32E
- renumbered J3 to J4
Connections:
- net GND: now reaches J4.1 (Pin_1)
- net GND: now also C49.2, U16.12 (~{G}), U16.14 (4A), U16.8 (GND)
- net EA+: now reaches J4.2 (Pin_2)
- net EA+: now also R30.2, U16.2 (1A)
- net EA-: now reaches J4.3 (Pin_3)
- net EA-: now also R30.1, U16.1 (1B)
- net EB+: now reaches J4.4 (Pin_4)
- net EB+: now also R29.1, U16.6 (2A)
- net EB-: now reaches J4.5 (Pin_5)
- net EB-: now also R29.2, U16.7 (2B)
- net EZ+: now reaches J4.6 (Pin_6)
- net EZ+: now also R28.2, U16.10 (3A)
- net EZ-: now reaches J4.7 (Pin_7)
- net EZ-: now also R28.1, U16.9 (3B)
- net +5V: now reaches J4.8 (Pin_8)
- new net +3V3: C49.1, U16.15 (4B), U16.16 (VDD), U16.4 (G)
- new net ENC_A: U16.3 (1Y)
- new net ENC_B: U16.5 (2Y)
- new net ENC_Z: U16.11 (3Y)
Other:
- company: (none) -> Doggen Engineering
- title: (none) -> Power Supply
- moved on the sheet: J4
