File: stm32u575ugtx.kicad_sch (KiCad schematic)
At the start: 39 parts, among them J5 TC2070, U12 STM32U575RGTx, U13 MCP2562-H-SN

Commit message: PCB Finished, only have to check LED's
Parts:
- removed C33: 100N-X7R_25V#0402, D&R_Passive:C_0402, symbol D&R_Passive:100N-X7R_25V#0402
- removed D9: BAT54C, Package_TO_SOT_SMD:SOT-23, symbol Diode:BAT54C
- added C34, C50, C51, C52, C53, C54, C55, C56: 100N-X7R_25V#0402, D&R_Passive:C_0402, symbol D&R_Passive:100N-X7R_25V#0402
- added J6: Conn_01x03, Connector_Phoenix_MC:PhoenixContact_MCV_1,5_3-G-3.81_1x03_P3.81mm_Vertical, symbol Connector_Generic:Conn_01x03
- added R32, R33, R34, R35, R36, R37, R38, R39, R68, R69, R70, R73, R82: 1K#0603, D&R_Passive:R_0603, symbol D&R_Passive:1K#0603
- added R62, R63, R64, R67, R72, R74, R75, R76, R77, R81: 10K#0603, D&R_Passive:R_0603, symbol D&R_Passive:10K#0603
- added R65: 150K#0603, D&R_Passive:R_0603, symbol D&R_Passive:150K#0603
- added R66, R71, R80: 33K#0603, D&R_Passive:R_0603, symbol D&R_Passive:33K#0603
- renumbered C31 to C24, C28 to C25, C34 to C26, C29 to C27, C30 to C28, C20 to C29, C21 to C30, C22 to C31, C23 to C32, C32 to C33, D8 to D4, D3 to D5, D4 to D6, D5 to D7, D2 to D8, R23 to R12, R15 to R13, R12 to R14, R16 to R15, R25 to R16, R14 to R17, R7 to R19, R26 to R20, R17 to R21, R13 to R22, R27 to R23, R19 to R24, R20 to R25, R21 to R26, R22 to R27, S3 to S2, S2 to S3, U12 to U14
Connections:
- net +3V3: now also R71.1, R74.1, R76.1
- net GND: now also C34.2, C50.2, C51.2, C52.2, C53.2, C54.2, C55.2, C56.2, J6.1 (Pin_1), R62.2, R63.2, R64.2, R72.2, R75.2, R77.2, R81.2
- net LED_BLUE: now also U14.39 (PC8)
- net LED_GRN: now also U14.44 (PA11)
- net LED_ORANGE: now also U14.43 (PA10)
- net LED_RED: now also U14.40 (PC9)
- net S0: now also U14.51 (PC10), R32.1; no longer S3.A9 (COM_9)
- net S1: now also U14.52 (PC11), R33.1; no longer S3.A8 (COM_8)
- net S2: now also U14.53 (PC12), R34.1; no longer S3.A7 (COM_7)
- net S3: now also U14.54 (PD2), R35.1; no longer S3.A6 (COM_6)
- net S4: now also U14.57 (PB5), R36.1; no longer S3.A5 (COM_5)
- net S5: now also U14.58 (PB6), R37.1; no longer S3.A4 (COM_4)
- net S6: now also U14.59 (PB7), R38.1; no longer S3.A3 (COM_3)
- net S7: now also U14.2 (PC13), R39.1; no longer S3.A2 (COM_2)
- net at R16.1: now also U14.21 (PA5); no longer U14.15 (PA1)
- net ADC4_IN3_5V: now reaches U14.10 (PC2)
- net ADC4_IN3_5V: now also C51.1, R70.2
- net ADC4_IN4_BOARD: now reaches U14.11 (PC3)
- net ADC4_IN4_BOARD: now also C54.1, R76.2, R77.1
- net REFL_OUT: now reaches U14.14 (PA0)
- net at U14.20 (PA4): no longer R20.1
- net ADC4_IN22_REV: now reaches U14.24 (PC4)
- net ADC4_IN22_REV: now also C52.1, R71.2, R72.1
- net ADC4_IN23_ASSY: now reaches U14.25 (PC5)
- net ADC4_IN23_ASSY: now also C53.1, R74.2, R75.1
- net at U14.26 (PB0): now also R20.1
- net at U14.27 (PB1): now also C55.1, R73.1
- net TMC5160_EN: now reaches U14.28 (PB2)
- net REF_SW: now reaches U14.3 (PC14)
- net REF_SW: now also C56.1, R82.2
- net 48V_EN: now reaches U14.38 (PC7)
- net ENC_A: now reaches U14.41 (PA8)
- net ENC_B: now reaches U14.42 (PA9)
- net ENC_Z: now reaches U14.45 (PA12)
- net ADC4_IN1_48V: now reaches U14.8 (PC0)
- net ADC4_IN1_48V: now also C34.1, R68.2
- net ADC4_IN2_12V: now reaches U14.9 (PC1)
- net ADC4_IN2_12V: now also C50.1, R69.2
- new net: R36.2, S3.A5 (COM_5)
- new net: R35.2, S3.A6 (COM_6)
- new net: R63.1, R66.2, R69.1
- new net: R80.2, R81.1, R82.1
- new net: R33.2, S3.A8 (COM_8)
- new net: R37.2, S3.A4 (COM_4)
- new net: R64.1, R67.2, R70.1
- new net: R32.2, S3.A9 (COM_9)
- new net: R62.1, R65.2, R68.1
- new net: J6.2 (Pin_2), R80.1
- new net: R34.2, S3.A7 (COM_7)
- new net: R38.2, S3.A3 (COM_3)
- new net: R39.2, S3.A2 (COM_2)
- new net +12V: J6.3 (Pin_3), R66.1
- new net +48V: R65.1
- new net +5V: R67.1
- new net 48V_VIOUT: R73.2
- new net REFR_OUT: U14.15 (PA1)
Other:
- note added: "* put these close to pins 1, 19, 32, 64, 48 respectively"
- note added: "8: 8x GPI dipswitch * 2: 1x UART naar TC2070 4: 4x Status LEDs (GPO) green, orange, red, blue * 4: SPI naar TMC5160 * 4: JTAG interface * 2: CAN Interface * 3: ADC psu measurement (5V, 12V, 48V) 3: ADC Rev. measurement (boardtype, hwrev, assy) 1: ADC ACS725 current sensor 1: 48V Softstart control line GPO * 3: Encoder A, B, Z (GPI inputs, quadrature encoder input/ timer? ) 1: Endstop switch (GPI)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"
- note added: "PSU ADC"
- note added: "REF SW"
- note removed: "* put these close to pins 1, 19, 32, 64, 13, 48 respectively"
- note removed: "8: 8x GPI dipswitch 4: 2x UART naar TC2070 4: 4x Status LEDs (GPO) green, orange, red, blue * 4: SPI naar TMC5160 * 4: JTAG interface 2: I2C Temp sensor * 2: CAN Interface 4: ADC psu measurement (3V3, 5V, 12V, 48V) 3: ADC Rev. measurement (boardtype, hwrev, assy) 1: ADC ACS725 current sensor 1: 48V Softstart control line GPO 3: Encoder A, B, Z (GPI inputs, quadrature encoder input/ timer? ) 1: En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"
- note removed: "PSU Measurement (ADC Protection)"
- company: (none) -> Doggen Engineering
- title: (none) -> Power Supply
- moved on the sheet: C25, C26, R14, R16, R20, R22, S1, S2
